File: cleanbot.kicad_pcb (KiCad board)
At the start: 2 copper layers, 85 x 56 mm, 65 parts, among them J1 MOTOR_L, J10 LINE_LED, J11 DXL_CONN, J12 CDC, J13 Cooling Fan, J14 ST Link, J15 NRST, J2 MOTOR_R, J3 SUCTION_MOTOR, J4 BATT_JACK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

Commit message: 두번째 버전
Parts:
- removed D7: BZT52Bxx, Diode_SMD:D_SOD-123F
- added C16: 20pF, Capacitor_SMD:C_0603_1608Metric_Pad1.08x0.95mm_HandSolder, F.Cu at (15.9, -23.1)
- added C17: 100nF, Capacitor_SMD:C_0603_1608Metric_Pad1.08x0.95mm_HandSolder, F.Cu at (71.4, -4.95)
- added C18: 100nF, Capacitor_SMD:C_0603_1608Metric_Pad1.08x0.95mm_HandSolder, B.Cu at (29.7, -26.5)
- added C19: 100nF, Capacitor_SMD:C_0603_1608Metric_Pad1.08x0.95mm_HandSolder, B.Cu at (41.0, -5.13)
- added C20: 100nF, Capacitor_SMD:C_0603_1608Metric_Pad1.08x0.95mm_HandSolder, B.Cu at (41.0, -11.2)
- added C21: 100nF, Capacitor_SMD:C_0603_1608Metric_Pad1.08x0.95mm_HandSolder, B.Cu at (41.0, -17.1)
- added C22: 100nF, Capacitor_SMD:C_0603_1608Metric_Pad1.08x0.95mm_HandSolder, B.Cu at (21.3, -47.8)
- added J16: SW1, Connector_Molex:Molex_SPOX_5267-02A_1x02_P2.50mm_Vertical, F.Cu at (39.4, -3.16)
- added J17: SW2, Connector_Molex:Molex_SPOX_5267-02A_1x02_P2.50mm_Vertical, F.Cu at (39.4, -9.13)
- added J18: SW3, Connector_Molex:Molex_SPOX_5267-02A_1x02_P2.50mm_Vertical, F.Cu at (39.4, -15.1)
- added R16: 10k, Resistor_SMD:R_0603_1608Metric_Pad0.98x0.95mm_HandSolder, B.Cu at (41.0, -12.8)
- added R17: 10k, Resistor_SMD:R_0603_1608Metric_Pad0.98x0.95mm_HandSolder, B.Cu at (41.0, -18.7)
- added R18: 0, Resistor_SMD:R_0603_1608Metric_Pad0.98x0.95mm_HandSolder, B.Cu at (21.8, -44.8)
- added R19: 0, Resistor_SMD:R_0603_1608Metric_Pad0.98x0.95mm_HandSolder, B.Cu at (16.1, -45.6)
- added R20: 10k, Resistor_SMD:R_0603_1608Metric_Pad0.98x0.95mm_HandSolder, B.Cu at (17.4, -48.8)
- added R21: 10k, Resistor_SMD:R_0603_1608Metric_Pad0.98x0.95mm_HandSolder, F.Cu at (55.5, -9.14)
- added U4: STM32F103RCTx, Package_QFP:LQFP-64_10x10mm_P0.5mm, F.Cu at (26.4, -34.3)
- added U5: 74LVC2G241, Package_SO:TSSOP-8_3x3mm_P0.65mm, F.Cu at (22.0, -45.2)
- C6: value 20pF -> 1uF
- J12: value CDC -> USB
- R13: value 10k -> 2.2k
- R14: value 160 -> 10k; moved to B.Cu
- R2: value 0 -> 10k
- U1: value STM32F103C8Tx -> CP2102N-Axx-xQFN28; footprint Package_QFP:LQFP-48_7x7mm_P0.5mm -> Package_DFN_QFN:QFN-28-1EP_5x5mm_P0.5mm_EP3.35x3.35mm
- moved C6 56.0 mm to (73.0, -4.95), turned to -90 degrees
- moved R2 47.4 mm to (74.8, -8.28), turned to 90 degrees
- moved U1 43.5 mm to (70.4, -10.2)
- moved R13 30.6 mm to (50.4, -36.2)
- moved C7 22.2 mm to (17.5, -36.4), turned to 90 degrees
- moved R1 12.1 mm to (13.5, -40.0), turned to 180 degrees
- moved C10 10.4 mm to (36.3, -32.1), turned to -90 degrees
- moved D5 7.44 mm to (44.3, -24.1)
- moved R11 7.34 mm to (44.3, -27.7)
- moved C3 7.29 mm to (26.4, -33.1), turned to 0 degrees
- moved Y1 7.09 mm to (17.2, -27.5)
- moved C5 6.41 mm to (26.4, -35.7), turned to 0 degrees
- moved C4 4.60 mm to (12.8, -26.2)
- moved C9 4.19 mm to (29.3, -42.5), turned to -45 degrees
- moved J6 4.19 mm to (80.0, -18.0)
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Connections:
- C6 pad 1: Net-(C6-Pad1) -> +5V
- J12 pad 1: unconnected-(J12-Pad1) -> +5V
- J13 pad 1: +5V -> RPI_5V
- J7 pad 1: +5V -> RPI_5V
- J9 pad 1: +5V -> RPI_5V
- R13 pad 1: Net-(D7-Pad1) -> /MOTOR_EN
- R13 pad 2: /DXL_UART -> GND
- R14 pad 1: 5V_Reg_out -> /SW1
- R14 pad 2: Net-(D7-Pad1) -> GND
- R2 pad 1: Net-(R2-Pad1) -> +5V
- R2 pad 2: Net-(C6-Pad1) -> Net-(R2-Pad2)
- U1 pad 1: +3V3 -> unconnected-(U1-Pad1)
- U1 pad 10: /MOTOR_PWM_L -> unconnected-(U1-Pad10)
- U1 pad 11: /MOTOR_PWM_R -> unconnected-(U1-Pad11)
- U1 pad 12: /MOTOR_DIR_L -> unconnected-(U1-Pad12)
- U1 pad 13: /MOTOR_DIR_R -> unconnected-(U1-Pad13)
- U1 pad 14: /MOTOR_EN -> unconnected-(U1-Pad14)
- U1 pad 15: /SUCTION_SIG -> unconnected-(U1-Pad15)
- U1 pad 16: /BUZZER_PWM -> unconnected-(U1-Pad16)
- U1 pad 18: /BATT_PWR_ADC -> unconnected-(U1-Pad18)
- U1 pad 19: /CURRENT_SENSE_ADC -> unconnected-(U1-Pad19)
- U1 pad 2: /PWR_BAD_LED -> unconnected-(U1-Pad2)
- U1 pad 23: GND -> unconnected-(U1-Pad23)
- U1 pad 24: +3V3 -> unconnected-(U1-Pad24)
- U1 pad 25: unconnected-(U1-Pad25) -> /UART1_TX
- U1 pad 26: unconnected-(U1-Pad26) -> /UART1_RX
- U1 pad 29: /MOTOR_PLS_L -> GND
- U1 pad 3: /PWR_NORM_LED -> GND
- U1 pad 4: /PWR_GOOD_LED -> /USBD+
- U1 pad 5: Net-(C4-Pad1) -> /USBD-
- U1 pad 6: Net-(R2-Pad1) -> /3.3V
- U1 pad 7: /NRST -> +5V
- U1 pad 8: GND -> +5V
- U1 pad 9: +3V3 -> Net-(R2-Pad2)
- Y1 pad 1: Net-(C6-Pad1) -> Net-(C16-Pad1)
Routing:
- net GND: track 114.4 -> 23.3 mm, vias 204 -> 17
- net +5V: track 19.0 -> 104.4 mm, vias 0 -> 8
- net /UART1_RX: track 0.00 -> 65.5 mm, vias 0 -> 2
- net /UART1_TX: track 0.00 -> 65.1 mm, vias 0 -> 2
- net /USBD-: track 74.0 -> 21.2 mm, vias 4 -> 2
- net /USBD+: track 75.1 -> 23.7 mm, vias 4 -> 2
- net /SW1: track 0.00 -> 40.1 mm, vias 0 -> 1
- net /SW2: track 0.00 -> 35.2 mm, vias 0 -> 1
- net /SW3: track 0.00 -> 33.7 mm, vias 0 -> 1
- net /PWR_GOOD_LED: track 46.0 -> 26.6 mm, vias 4 -> 0
- net RPI_5V: track 0.00 -> 19.0 mm
- net /DXL_UART_TX: track 0.00 -> 17.2 mm, vias 0 -> 4
- net /DXL_UART_RX: track 0.00 -> 15.7 mm, vias 0 -> 3
- net +3V3: track 145.3 -> 159.9 mm, vias 17 -> 16
- net /BATT_PWR_ADC: track 34.9 -> 48.0 mm
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Other:
- board text added: "2022 GSR Cleanbot ver.2 by LSH"
- board text removed: "2022 GSR Cleanbot ver.1"
