File: cleanbot.kicad_sch (KiCad schematic)
At the start: 61 parts, among them J1 MOTOR_L, J10 LINE_LED, J11 DXL_CONN, J12 CDC, J13 Cooling Fan, J14 ST Link, J15 NRST, J2 MOTOR_R, J3 SUCTION_MOTOR, J4 BATT_JACK, J5 12V_OUT, J6 5V_IN, J7 RPI_PWR, J8 PWR_sw, J9 RPI_sw, Q1 IRLML6244, Q2 KRC106S, U1 STM32F103C8Tx, U2 LD1117S33TR_SOT223, U3 INA240A3D, Y1 8MHz

Commit message: 두번째 버전
Parts:
- removed D7: BZT52Bxx, Diode_SMD:D_SOD-123F, symbol Diode:BZT52Bxx
- removed U1: STM32F103C8Tx, Package_QFP:LQFP-48_7x7mm_P0.5mm, symbol MCU_ST_STM32F1:STM32F103C8Tx
- added C16: 20pF, Capacitor_SMD:C_0603_1608Metric_Pad1.08x0.95mm_HandSolder, symbol Device:C
- added C17, C18, C19, C20, C21, C22: 100nF, Capacitor_SMD:C_0603_1608Metric_Pad1.08x0.95mm_HandSolder, symbol Device:C
- added J16: SW1, Connector_Molex:Molex_SPOX_5267-02A_1x02_P2.50mm_Vertical, symbol Connector:Conn_01x02_Female
- added J17: SW2, Connector_Molex:Molex_SPOX_5267-02A_1x02_P2.50mm_Vertical, symbol Connector:Conn_01x02_Female
- added J18: SW3, Connector_Molex:Molex_SPOX_5267-02A_1x02_P2.50mm_Vertical, symbol Connector:Conn_01x02_Female
- added R16, R17, R20, R21: 10k, Resistor_SMD:R_0603_1608Metric_Pad0.98x0.95mm_HandSolder, symbol Device:R
- added R18, R19: 0, Resistor_SMD:R_0603_1608Metric_Pad0.98x0.95mm_HandSolder, symbol Device:R
- added U1: CP2102N-Axx-xQFN28, Package_DFN_QFN:QFN-28-1EP_5x5mm_P0.5mm_EP3.35x3.35mm, symbol Interface_USB:CP2102N-Axx-xQFN28
- added U4: STM32F103RCTx, Package_QFP:LQFP-64_10x10mm_P0.5mm, symbol MCU_ST_STM32F1:STM32F103RCTx
- added U5: 74LVC2G241, Package_SO:TSSOP-8_3x3mm_P0.65mm, symbol 74xGxx:74LVC2G241
- C6: value 20pF -> 1uF
- J12: value CDC -> USB
- R13: value 10k -> 2.2k
- R14: value 160 -> 10k
- R2: value 0 -> 10k
Connections:
- net +3V3: now also C18.1, C19.1, C20.1, C21.1, J16.1 (Pin_1), J17.1 (Pin_1), J18.1 (Pin_1), U4.1 (VBAT), U4.13 (VDDA), U4.19 (VDD), U4.32 (VDD), U4.48 (VDD), U4.64 (VDD)
- net +5V: now also C6.1, J12.1 (VBUS), R2.1, C22.1, R20.1, R21.1, U1.7 (VREGIN), U1.8 (VBUS), U5.8 (VCC), U5.8 (VCC); no longer J13.1 (Pin_1), J7.1 (Pin_1), J9.1 (Pin_1)
- net 5V_Reg_out: no longer R14.1
- net BATT_PWR_ADC: now also U4.24 (PC4)
- net BUZZER_PWM: now also U4.37 (PC6)
- net CURRENT_SENSE_ADC: now also U4.25 (PC5)
- net DXL_UART: now also R21.2, U5.2, U5.3; no longer R13.2
- net GND: now also R13.2, R14.2, C16.2, C17.2, C18.2, C22.2, R16.2, R17.2, U1.29 (GND), U1.3 (GND), U4.12 (VSSA), U4.18 (VSS), U4.31 (VSS), U4.47 (VSS), U4.63 (VSS), U5.4 (GND), U5.4 (GND)
- net MOTOR_DIR_L: now also U4.21 (PA5)
- net MOTOR_DIR_R: now also U4.22 (PA6)
- net MOTOR_EN: now also R13.1, U4.20 (PA4)
- net MOTOR_PLS_L: now also U4.29 (PB10)
- net MOTOR_PLS_R: now also U4.30 (PB11)
- net MOTOR_PWM_L: now also U4.41 (PA8)
- net MOTOR_PWM_R: now also U4.42 (PA9)
- net NRST: now also U4.7 (NRST)
- net PWR_BAD_LED: now also U4.2 (PC13)
- net PWR_GOOD_LED: now also U4.4 (PC15)
- net PWR_NORM_LED: now also U4.3 (PC14)
- net SUCTION_SIG: now also U4.26 (PB0)
- net SWCLK: now also U4.49 (PA14)
- net SWDIO: now also U4.46 (PA13)
- net USBD+: now also U1.4 (D+)
- net USBD-: now also U1.5 (D-)
- net at R1.1: now also U4.60 (BOOT0)
- net at C4.1, Y1.2: now also U4.5 (PD0)
- new net: R18.2, R19.2, U5.1, U5.7
- new net: C16.1, U4.6 (PD1), Y1.1
- new net: R2.2, U1.9 (~{RST})
- new net 3.3V: C17.1, U1.6 (VDD)
- new net DXL_TX_EN: R18.1, U4.50 (PA15)
- new net DXL_UART_RX: R20.2, U4.52 (PC11), U5.6
- new net DXL_UART_TX: R19.1, U4.51 (PC10), U5.5
- new net RPI_5V: J13.1 (Pin_1), J7.1 (Pin_1), J9.1 (Pin_1)
- new net SW1: C19.2, J16.2 (Pin_2), R14.1, U4.8 (PC0)
- new net SW2: C20.2, J17.2 (Pin_2), R16.1, U4.9 (PC1)
- new net SW3: C21.2, J18.2 (Pin_2), R17.1, U4.10 (PC2)
- new net UART1_RX: U1.26 (TXD), U4.59 (PB7)
- new net UART1_TX: U1.25 (RXD), U4.58 (PB6)
- no-connect marks 19 -> 45
Other:
- note added: "Dynamixel"
- note added: "EXT. Switches"
- note added: "USB VCP"
- note removed: "5.1V zener"
- note removed: "Dynamixel Connector"
- note removed: "USB CDC Connector"
- moved on the sheet: C1, C10, C11, C12, C13, C14, C15, C2, C3, C5, C7, C8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
